File: eog-pcb-kicad/eog-pcb-kicad.kicad_sch (KiCad schematic)
At the start: 101 parts, among them J1 Conn_01x03, J2 Conn_01x02, J3 Conn_01x02, J4 Conn_01x03, J6 Conn_01x02, U2 AD620, U3 LMC6482, U4 LMC6482, U5 AD620, U6 LMC6482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

Commit message: added libraries for digipots and started reorganizing the pcb for 2nd version
Parts:
- removed R10: 100k, Resistor_SMD:R_0603_1608Metric, symbol Device:R_US
- removed R23, R8: 10k, Resistor_SMD:R_0603_1608Metric, symbol Device:R_US
- removed R4, R5: 320R, Resistor_SMD:R_0603_1608Metric, symbol Device:R_US
- removed R9: 150R, Resistor_SMD:R_0603_1608Metric, symbol Device:R_US
- added U1, U11: AD8402ARZ1, Package_SO:SOIC-14_3.9x8.7mm_P1.27mm, symbol AD8402ARZ1:AD8402ARZ1
- added U10, U13: MAX5401EKAT, Package_TO_SOT_SMD:SOT-23-8, symbol MAX5401EKAT:MAX5401EKAT
- added U12, U9: AD5160BRJZ5-RL7, Package_TO_SOT_SMD:SOT-23-8, symbol AD5160BRJZ5-RL7:AD5160BRJZ5-RL7
- U2, U5: footprint Package_DIP:DIP-8_W7.62mm -> Package_SO:SOIC-8_3.9x4.9mm_P1.27mm
- U8: footprint SOIC127P600X175-8N -> Package_SO:SOIC-8_3.9x4.9mm_P1.27mm
Connections:
- net GND: now also U12.3 (GND), U12.7 (B), U9.3 (GND), U9.7 (B)
- net HPF_OUT_CH0: now also U9.1 (W)
- net HPF_OUT_CH1: now also U12.1 (W)
- net VDD: now also U12.2 (VDD), U12.8 (A), U9.2 (VDD), U9.8 (A)
Other:
- note added: "R4 and R5 here"
- note added: "R9 and R10 here"
- moved on the sheet: C13, C14, C15, C21, C22, C23, C3, C5, J3, R11, R12, R13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
