File: eog-pcb-kicad/eog-pcb-kicad.kicad_sch (KiCad schematic)
At the start: 108 parts, among them J1 INPUT0, J10 RG0, J11 RG1, J2 HPF0, J3 G0, J4 Conn_01x02, J5 Conn_01x02, J6 INPUT1, J7 HPF1, J8 G1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

Commit message: preliminary layout and added libraries
Parts:
- removed TP12, TP18: TestPoint, TestPoint:TestPoint_Pad_1.0x1.0mm, symbol Connector:TestPoint
- J5: value Conn_01x02 -> OUT0
- J9: value Conn_01x02 -> OUT1
- U5: footprint SOIC127P600X175-8N -> MAX764ESA_:SOIC127P600X175-8N
Changed lines of the file:
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@@
   (junction (at 278.892 271.78) (diameter 0) (color 0 0 0 0)
   )
-  (junction (at 381.889 328.041) (diameter 0) (color 0 0 0 0)
-  )
   (junction (at 271.399 327.66) (diameter 0) (color 0 0 0 0)
   )
@@
   (junction (at 376.047 328.041) (diameter 0) (color 0 0 0 0)
   )
-  (junction (at 56.5658 318.5414) (diameter 0) (color 0 0 0 0)
-  )
   (junction (at 249.809 330.2) (diameter 0) (color 0 0 0 0)
   )
@@
     (stroke (width 0) (type default) (color 0 0 0 0))
   )
-  (wire (pts (xy 381.889 328.041) (xy 384.81 328.041))
-    (stroke (width 0) (type default) (color 0 0 0 0))
-  )
   (polyline (pts (xy 272.923 307.467) (xy 272.923 358.775))
     (stroke (width 0.2) (type default) (color 0 0 0 0))
@@
     (stroke (width 0) (type default) (color 0 0 0 0))
   )
-  (wire (pts (xy 69.6468 318.5414) (xy 56.5658 318.5414))
-    (stroke (width 0) (type default) (color 0 0 0 0))
-  )
   (wire (pts (xy 56.5658 325.2724) (xy 67.1068 325.2724))
     (stroke (width 0) (type default) (color 0 0 0 0))
@@
       (effects (font (size 1.27 1.27)) (justify left))
     )
-    (property "Value" "Conn_01x02" (id 1) (at 75.1078 327.8123 0)
+    (property "Value" "OUT0" (id 1) (at 75.1078 327.8123 0)
       (effects (font (size 1.27 1.27)) (justify left))
     )
@@
     (pin "1")
   )
-  (symbol (lib_id "Connector:TestPoint") (at 384.81 328.041 270) (unit 1)
-    (in_bom yes) (on_board yes)
-    (property "Reference" "TP18" (id 0) (at 389.89 326.771 0)
-      (effects (font (size 1.27 1.27)) (justify left))
-    )
-    (property "Value" "TestPoint" (id 1) (at 386.8421 330.581 0)
-      (effects (font (size 1.27 1.27)) (justify left) hide)
-    )
-    (property "Footprint" "TestPoint:TestPoint_Pad_1.0x1.0mm" (id 2) (at 384.81 333.121 0)
-      (effects (font (size 1.27 1.27)) hide)
-    )
-    (property "Datasheet" "~" (id 3) (at 384.81 333.121 0)
-      (effects (font (size 1.27 1.27)) hide)
-    )
-    (pin "1")
-  )
   (symbol (lib_id "MBRS330T3G:MBRS330T3G") (at 172.339 54.991 180) (unit 1)
     (in_bom yes) (on_board yes)
@@
       (effects (font (size 1.27 1.27)) (justify left))
     )
-    (property "Value" "Conn_01x02" (id 1) (at 403.606 337.6929 0)
+    (property "Value" "OUT1" (id 1) (at 403.606 337.6929 0)
       (effects (font (size 1.27 1.27)) (justify left))
     )
@@
     (pin "2")
   )
-  (symbol (lib_id "Connector:TestPoint") (at 69.6468 318.5414 270) (unit 1)
-    (in_bom yes) (on_board yes)
-    (property "Reference" "TP12" (id 0) (at 74.7268 317.2714 0)
-      (effects (font (size 1.27 1.27)) (justify left))
-    )
-    (property "Value" "TestPoint" (id 1) (at 71.6789 321.0814 0)
-      (effects (font (size 1.27 1.27)) (justify left) hide)
-    )
-    (property "Footprint" "TestPoint:TestPoint_Pad_1.0x1.0mm" (id 2) (at 69.6468 323.6214 0)
-      (effects (font (size 1.27 1.27)) hide)
-    )
-    (property "Datasheet" "~" (id 3) (at 69.6468 323.6214 0)
-      (effects (font (size 1.27 1.27)) hide)
-    )
-    (pin "1")
-  )
   (symbol (lib_id "power:VDD") (at 232.156 102.3874 0) (unit 1)
     (in_bom yes) (on_board yes) (fields_autoplaced)
@@
     (property "Reference" "U5" (id 0) (at 139.065 42.164 0))
     (property "Value" "MAX764ESA+" (id 1) (at 139.065 44.704 0))
-    (property "Footprint" "SOIC127P600X175-8N" (id 2) (at 139.065 60.071 0)
+    (property "Footprint" "MAX764ESA_:SOIC127P600X175-8N" (id 2) (at 139.065 60.071 0)
       (effects (font (size 1.27 1.27)) (justify left bottom) hide)
     )
@@
     )
     (path "/008f06b1-976d-4955-bd87-d80bc72e31b6"
-      (reference "J5") (unit 1) (value "Conn_01x02") (footprint "Connector_PinHeader_2.54mm:PinHeader_1x02_P2.54mm_Vertical")
+      (reference "J5") (unit 1) (value "OUT0") (footprint "Connector_PinHeader_2.54mm:PinHeader_1x02_P2.54mm_Vertical")
     )
     (path "/41cdcb08-897d-4955-87ea-d0f5b7f9819c"
@@
     )
     (path "/1040cdd9-6558-48f6-9533-38c30b778f55"
-      (reference "J9") (unit 1) (value "Conn_01x02") (footprint "Connector_PinHeader_2.54mm:PinHeader_1x02_P2.54mm_Vertical")
+      (reference "J9") (unit 1) (value "OUT1") (footprint "Connector_PinHeader_2.54mm:PinHeader_1x02_P2.54mm_Vertical")
     )
     (path "/94f8e1b5-4d9d-48ba-b7ba-1c7bf0b4438d"
@@
       (reference "TP11") (unit 1) (value "TestPoint") (footprint "TestPoint:TestPoint_Pad_1.0x1.0mm")
     )
-    (path "/de086212-f71e-4467-97af-4e551c4d43fa"
-      (reference "TP12") (unit 1) (value "TestPoint") (footprint "TestPoint:TestPoint_Pad_1.0x1.0mm")
-    )
     (path "/347f5700-9a09-46e4-a110-37c9b7d87523"
       (reference "TP13") (unit 1) (value "TestPoint") (footprint "TestPoint:TestPoint_Pad_1.0x1.0mm")
@@
       (reference "TP17") (unit 1) (value "TestPoint") (footprint "TestPoint:TestPoint_Pad_1.0x1.0mm")
     )
-    (path "/06130db8-5d12-446b-a1fc-9109ad697443"
-      (reference "TP18") (unit 1) (value "TestPoint") (footprint "TestPoint:TestPoint_Pad_1.0x1.0mm")
-    )
     (path "/fd204c06-7578-4b62-ae76-1989b9f0bab1"
       (reference "TP19") (unit 1) (value "TestPoint") (footprint "TestPoint:TestPoint_Pad_1.0x1.0mm")
@@
     )
     (path "/e7c2fa04-5da8-4510-86af-c81dc93e39fb"
-      (reference "U5") (unit 1) (value "MAX764ESA+") (footprint "SOIC127P600X175-8N")
+      (reference "U5") (unit 1) (value "MAX764ESA+") (footprint "MAX764ESA_:SOIC127P600X175-8N")
     )
     (path "/0851747f-c938-492c-92cf-a1bee970415e"
