File: eog-pcb-kicad/_autosave-eog-pcb-kicad.kicad_sch (KiCad schematic)
At the start: 95 parts, among them J1 Conn_01x03, J2 Conn_01x12, J4 Conn_01x03, U1 AD8402ARZ1, U10 MAX5401EKAT, U11 AD8402ARZ1, U12 AD5160BRJZ5-RL7, U13 MAX5401EKAT, U2 AD620, U3 LMC6482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

Commit message: gen2 board is ready and production files are generated
Parts:
- removed J2: Conn_01x12, Connector_PinHeader_2.54mm:PinHeader_1x12_P2.54mm_Vertical, symbol Connector_Generic:Conn_01x12
- removed TP1, TP10, TP11, TP13, TP14, TP15, TP16, TP17, TP18, TP19, TP2, TP3, TP4, TP5, TP7, TP8, TP9: TestPoint, TestPoint:TestPoint_Pad_1.0x1.0mm, symbol Connector:TestPoint
- added J2: Conn_01x08, Connector_PinHeader_2.54mm:PinHeader_1x08_P2.54mm_Vertical, symbol Connector_Generic:Conn_01x08
- added J3: Conn_01x04, Connector_PinHeader_2.54mm:PinHeader_1x04_P2.54mm_Vertical, symbol Connector_Generic:Conn_01x04
- added LED1: LED, LED_SMD:LED_0603_1608Metric, symbol Device:LED
- added R5: 400, Resistor_SMD:R_0603_1608Metric, symbol Device:R_US
Connections:
- net AOUT_CH0: now also J3.3 (Pin_3)
- net AOUT_CH1: now also J3.2 (Pin_2)
- net CLK: now also J2.8 (Pin_8)
- net CS1: now also J2.1 (Pin_1)
- net CS2: now also J2.2 (Pin_2)
- net CS3: now also J2.3 (Pin_3)
- net CS4: now also J2.4 (Pin_4)
- net CS5: now also J2.5 (Pin_5)
- net CS6: now also J2.6 (Pin_6)
- net GND: now also J3.1 (Pin_1), LED1.1 (K)
- net SDI: now also J2.7 (Pin_7)
- net VDD: now also J3.4 (Pin_4), R5.1
- new net: LED1.2 (A), R5.2
Other:
- note added: "TODO: calculate resistor value based on LED specs"
- note removed: "TEST POINTS"

Commit message: updating BOM and CPL files
Parts:
- R5: value 400 -> 330R
Changed lines of the file:
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@@
       (effects (font (size 1.27 1.27)) (justify left))
     )
-    (property "Value" "400" (id 1) (at 198.12 134.8739 0)
+    (property "Value" "330R" (id 1) (at 198.12 134.8739 0)
       (effects (font (size 1.27 1.27)) (justify left))
     )
@@
     )
     (path "/1a74e4ef-9f04-445e-a4d4-879b5e2f061a"
-      (reference "R5") (unit 1) (value "400") (footprint "Resistor_SMD:R_0603_1608Metric")
+      (reference "R5") (unit 1) (value "330R") (footprint "Resistor_SMD:R_0603_1608Metric")
     )
     (path "/2f18daab-5439-4af5-81ac-008222e75137"
