File: eog-pcb-kicad/eog-pcb-kicad.kicad_pcb (KiCad board)
At the start: 4 copper layers, 60 x 41 mm, 82 parts, among them J1 Conn_01x03, J2 Conn_01x08, J3 Conn_01x04, J4 Conn_01x03, U1 AD8402ARZ1, U10 MAX5401EKAT, U11 AD8402ARZ1, U12 AD5160BRJZ5-RL7, U13 MAX5401EKAT, U2 AD620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

Commit message: updating BOM and CPL files
Parts:
- moved H3 3.50 mm to (56.5, 37.5)
Changed lines of the file:
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@@
       (layerselection 0x00010fc_ffffffff)
       (disableapertmacros false)
-      (usegerberextensions false)
+      (usegerberextensions true)
       (usegerberattributes true)
-      (usegerberadvancedattributes true)
-      (creategerberjobfile true)
+      (usegerberadvancedattributes false)
+      (creategerberjobfile false)
       (svguseinch false)
       (svgprecision 6)
@@
       (drillshape 0)
       (scaleselection 1)
-      (outputdirectory "")
+      (outputdirectory "../production/gerbers/")
     )
   )
@@
   )
   (footprint "MountingHole:MountingHole_2.2mm_M2" (layer "F.Cu")
-    (at 56.5 34)
+    (at 56.5 37.5)
     (descr "Mounting Hole 2.2mm, no annular, M2")
     (tags "mounting hole 2.2mm no annular m2")
